Commit message: add diffbot controllers

File: diffbot_description/urdf/diffbot.urdf.xacro (robot description, xacro)
@@ -1,4 +1,5 @@
 <?xml version="1.0"?>
 <robot name="diffbot" xmlns:xacro="http://ros.org/wiki/xacro">
+  <xacro:include filename="$(find diffbot_description)/urdf/diffbot_ros2_control.xacro" />
   <xacro:include filename="$(find diffbot_description)/urdf/diffbot_gazebo.xacro" />
   <xacro:include filename="$(find diffbot_description)/urdf/diffbot_material.xacro" />

File: diffbot_description/urdf/diffbot_gazebo.xacro (robot description, xacro)
@@ -1,4 +1,18 @@
-<?xml version="1.0" encoding="UTF-8"?>
+<?xml version="1.0"?>
 <robot name="diffbot" xmlns:xacro="http://ros.org/wiki/xacro">
+  <transmission name="wheel_right_transmission">
+    <plugin>transmission_interface/SimpleTransmission</plugin>
+    <actuator name="wheel_right_motor" role="actuator_right"/>
+    <joint name="wheel_right_joint"    role="joint_right">
+      <mechanical_reduction>1.0</mechanical_reduction>
+    </joint>
+  </transmission>
+  <transmission name="wheel_left_transmission">
+    <plugin>transmission_interface/SimpleTransmission</plugin>
+    <actuator name="wheel_left_motor" role="actuator_left"/>
+    <joint name="wheel_left_joint"    role="joint_left">
+      <mechanical_reduction>1.0</mechanical_reduction>
+    </joint>
+  </transmission>
   <gazebo reference="wheel_left_link">
     <mu1>1000000000000000.0</mu1>
@@ -36,3 +50,10 @@
     <maxVel>1.0</maxVel>
   </gazebo>
+  <gazebo>
+    <plugin filename="libgazebo_ros2_control.so" name="gazebo_ros2">
+      <robot_parm>robot_description</robot_parm>
+      <robot_parm_node>robot_state_publisher</robot_parm_node>
+      <parameters>$(find diffbot_controllers)/config/diffbot_controllers.yaml</parameters>
+    </plugin>
+  </gazebo>
 </robot>

Commit message: migration to gazebo fortress

File: diffbot_description/urdf/diffbot.urdf.xacro (robot description, xacro)
@@ -140,3 +140,28 @@
     <axis xyz="0 0 0" />
   </joint>
+  <!-- Hokuyo Laser -->
+  <link name="hokuyo_link">
+    <collision>
+      <origin xyz="0 0 0" rpy="0 0 0"/>
+      <geometry>
+    <box size="0.05 0.05 0.05"/>
+      </geometry>
+    </collision>
+    <visual>
+      <origin xyz="0 0 0" rpy="0 0 0"/>
+      <geometry>
+        <mesh filename="package://diffbot_description/meshes/hokuyo.dae"/>
+      </geometry>
+    </visual>
+    <inertial>
+      <mass value="1e-5" />
+      <origin xyz="0 0 0" rpy="0 0 0"/>
+      <inertia ixx="1e-6" ixy="0" ixz="0" iyy="1e-6" iyz="0" izz="1e-6" />
+    </inertial>
+  </link>
+  <joint name="hokuyo_joint" type="fixed">
+    <origin xyz="0 0 0.11" rpy="0 0 0"/>
+    <parent link="base_link"/>
+    <child link="hokuyo_link"/>
+  </joint>
 </robot>

File: diffbot_description/urdf/diffbot_gazebo.xacro (robot description, xacro)
@@ -3,6 +3,6 @@
   <transmission name="wheel_right_transmission">
     <plugin>transmission_interface/SimpleTransmission</plugin>
-    <actuator name="wheel_right_motor" role="actuator_right"/>
-    <joint name="wheel_right_joint"    role="joint_right">
+    <actuator name="wheel_right_motor" role="actuator_right" />
+    <joint name="wheel_right_joint" role="joint_right">
       <mechanical_reduction>1.0</mechanical_reduction>
     </joint>
@@ -10,6 +10,6 @@
   <transmission name="wheel_left_transmission">
     <plugin>transmission_interface/SimpleTransmission</plugin>
-    <actuator name="wheel_left_motor" role="actuator_left"/>
-    <joint name="wheel_left_joint"    role="joint_left">
+    <actuator name="wheel_left_motor" role="actuator_left" />
+    <joint name="wheel_left_joint" role="joint_left">
       <mechanical_reduction>1.0</mechanical_reduction>
     </joint>
@@ -33,5 +33,4 @@
     <fdir1>1 0 0</fdir1>
   </gazebo>
-  <!-- Caster Wheels -->
   <gazebo reference="caster_rear_link">
     <mu1>0.1</mu1>
@@ -51,5 +50,6 @@
   </gazebo>
   <gazebo>
-    <plugin filename="libgazebo_ros2_control.so" name="gazebo_ros2">
+    <plugin filename="libgz_ros2_control-system.so"
+      name="gz_ros2_control::GazeboSimROS2ControlPlugin">
       <robot_parm>robot_description</robot_parm>
       <robot_parm_node>robot_state_publisher</robot_parm_node>

File: diffbot_description/urdf/diffbot_ros2_control.xacro (robot description, xacro)
@@ -1,7 +1,7 @@
 <?xml version="1.0"?>
 <robot name="diffbot" xmlns:xacro="http://ros.org/wiki/xacro">
-  <ros2_control type="system" name="RobotSystem">
+  <ros2_control name="GazeboSimSystem" type="system">
     <hardware>
-      <plugin>gazebo_ros2_control/GazeboSystem</plugin>
+      <plugin>gz_ros2_control/GazeboSimSystem</plugin>
     </hardware>
     <joint name="wheel_left_joint">

Commit message: add lidar sensor

File: diffbot_description/urdf/diffbot.urdf.xacro (robot description, xacro)
@@ -4,5 +4,5 @@
   <xacro:include filename="$(find diffbot_description)/urdf/diffbot_gazebo.xacro" />
   <xacro:include filename="$(find diffbot_description)/urdf/diffbot_material.xacro" />
-  <link name="base_footprint"/>
+  <link name="world"/>
   <link name="base_link">
     <inertial>
@@ -27,5 +27,5 @@
   </link>
   <joint name="base_joint" type="fixed">
-    <parent link="base_footprint"/>
+    <parent link="world"/>
     <child link="base_link" />
     <origin xyz="0 0 0.033" rpy="0 0 0"/>
@@ -140,28 +140,30 @@
     <axis xyz="0 0 0" />
   </joint>
-  <!-- Hokuyo Laser -->
-  <link name="hokuyo_link">
+  <link name="laser_link">
+    <inertial>
+      <origin xyz="-0.011945780406062 -0.000381929217680526 -0.0170649378129477" rpy="0 0 0" />
+      <mass value="0.073084435549317" />
+      <inertia ixx="1.96074931730795E-05" ixy="-3.62091076640009E-07" ixz="4.28230084046735E-07"
+               iyy="2.40983835136327E-05" iyz="1.50180909250652E-08"
+               izz="4.14184164228595E-05" />
+    </inertial>
+    <visual>
+      <origin xyz="0 0 0" rpy="0 0 0" />
+      <geometry>
+        <mesh filename="package://diffbot_description/meshes/laser_link.STL" />
+      </geometry>
+    </visual>
     <collision>
-      <origin xyz="0 0 0" rpy="0 0 0"/>
+      <origin xyz="0 0 0" rpy="0 0 0" />
       <geometry>
-    <box size="0.05 0.05 0.05"/>
+        <mesh filename="package://diffbot_description/meshes/laser_link.STL" />
       </geometry>
     </collision>
-    <visual>
-      <origin xyz="0 0 0" rpy="0 0 0"/>
-      <geometry>
-        <mesh filename="package://diffbot_description/meshes/hokuyo.dae"/>
-      </geometry>
-    </visual>
-    <inertial>
-      <mass value="1e-5" />
-      <origin xyz="0 0 0" rpy="0 0 0"/>
-      <inertia ixx="1e-6" ixy="0" ixz="0" iyy="1e-6" iyz="0" izz="1e-6" />
-    </inertial>
   </link>
-  <joint name="hokuyo_joint" type="fixed">
-    <origin xyz="0 0 0.11" rpy="0 0 0"/>
-    <parent link="base_link"/>
-    <child link="hokuyo_link"/>
+  <joint name="laser_joint" type="fixed">
+    <origin xyz="-0.0050526 -0.0023221 0.1208" rpy="0 0 0" />
+    <parent link="base_link" />
+    <child link="laser_link" />
+    <axis xyz="0 0 1" />
   </joint>
 </robot>

File: diffbot_description/urdf/diffbot_gazebo.xacro (robot description, xacro)
@@ -88,4 +88,33 @@
     </sensor>
   </gazebo>
+  <gazebo reference="laser_link">
+    <sensor name="lidar" type="gpu_lidar">
+      <ign_frame_id>laser_link</ign_frame_id>
+      <always_on>true</always_on>
+      <visualize>true</visualize>
+      <topic>scan</topic>
+      <update_rate>5</update_rate>
+      <lidar>
+        <scan>
+          <horizontal>
+            <samples>360</samples>
+            <resolution>1.00000</resolution>
+            <min_angle>0.000000</min_angle>
+            <max_angle>6.280000</max_angle>
+          </horizontal>
+        </scan>
+        <range>
+          <min>0.120000</min>
+          <max>12.0</max>
+          <resolution>0.02</resolution>
+        </range>
+        <noise>
+          <type>gaussian</type>
+          <mean>0.0</mean>
+          <stddev>0.01</stddev>
+        </noise>
+      </lidar>
+    </sensor>
+  </gazebo>
   <gazebo>
     <plugin filename="libgz_ros2_control-system.so"

Commit message: change name of base frame

File: diffbot_description/urdf/diffbot.urdf.xacro (robot description, xacro)
@@ -4,5 +4,5 @@
   <xacro:include filename="$(find diffbot_description)/urdf/diffbot_gazebo.xacro" />
   <xacro:include filename="$(find diffbot_description)/urdf/diffbot_material.xacro" />
-  <link name="world"/>
+  <link name="base_footprint"/>
   <link name="base_link">
     <inertial>
@@ -27,5 +27,5 @@
   </link>
   <joint name="base_joint" type="fixed">
-    <parent link="world"/>
+    <parent link="base_footprint"/>
     <child link="base_link" />
     <origin xyz="0 0 0.033" rpy="0 0 0"/>
